File: mk3/SMD.brd (EAGLE design)
At the start: 31.3 x 39 mm, 13 parts, among them IC1 744053D

Commit message: Changed base resistor to 1k.
Parts:
- R3: value 330 -> 1K
Changed lines of the file:
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@@
 <attribute name="VALUE" x="6.50875" y="25.55875" size="1.27" layer="27" rot="R90"/>
 </element>
-<element name="R3" library="rcl" package="M1206" value="330" x="7.46125" y="27.94" smashed="yes" rot="R90">
+<element name="R3" library="rcl" package="M1206" value="1K" x="7.46125" y="27.94" smashed="yes" rot="R90">
 <attribute name="VALUE" x="7.46125" y="27.94" size="0.8128" layer="27" font="vector" rot="R90" align="center"/>
 </element>
