File: mk3/THT.brd (EAGLE design)
At the start: 31.3 x 44 mm, 13 parts, among them IC1 74HC4053P

Commit message: Changed base resistor to 1k.
Parts:
- R3: value 330 -> 1K
Changed lines of the file:
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@@
 <attribute name="VALUE" x="5.23875" y="30.63875" size="1.27" layer="27" rot="R90"/>
 </element>
-<element name="R3" library="rcl" package="0207/2V" value="330" x="2.54" y="27.84" smashed="yes" rot="R180"/>
+<element name="R3" library="rcl" package="0207/2V" value="1K" x="2.54" y="27.84" smashed="yes" rot="R180"/>
 <element name="JP2" library="jumper" package="JP2" value="" x="1.905" y="39.859528125" smashed="yes" rot="SR90">
 <attribute name="NAME" x="4.553528125" y="36.576" size="1.27" layer="25" ratio="10" rot="SR0"/>
