File: mk3/SMD.sch (EAGLE design)
At the start: 13 parts, among them IC1 744053D

Commit message: Changed base resistor to 1k.
Parts:
- R3: value 330 -> 1K
Changed lines of the file:
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@@
 <part name="T1" library="transistor-neu-to92" deviceset="*-NPN-" device="SOT23-BEC" technology="MMBT3904LT1"/>
 <part name="P+2" library="supply1" deviceset="VCC" device=""/>
-<part name="R3" library="rcl" deviceset="R-EU_" device="M1206" value="330"/>
+<part name="R3" library="rcl" deviceset="R-EU_" device="M1206" value="1K"/>
 <part name="GND3" library="supply1" deviceset="GND" device=""/>
 </parts>

Commit message: CD4053
Parts:
- removed IC1: 744053D, 74xx-eu:744053D
- added U1: CD4053BCM, Fairchild_By_element14_Batch_1:CD4053BCM
Connections:
- removed net N$6: IC1G$1.3Y0, R9.S
- new net N$2: R7.S, U1.AX
- net GND: now also U1.INH, U1.VEE, U1.VSS; no longer IC1G$1.E, IC1P.GND, IC1P.VEE
- net MONOSIGNAL: now also U1.AY, U1.BY, U1.CY; no longer IC1G$1.1Y1, IC1G$1.2Y1, IC1G$1.3Y1
- net N$4: now also R8.S, U1.BX; no longer IC1G$1.1Y0, R7.S
- net N$5: now also R9.S, U1.CX; no longer IC1G$1.2Y0, R8.S
- net SELECT: now also U1.A_2, U1.B_2, U1.C; no longer IC1G$1.S1, IC1G$1.S2, IC1G$1.S3
- net VBLUE: now also U1.0; no longer IC1G$1.3Z
- net VCC: now also U1.VDD
- net VGREEN: now also U1.B; no longer IC1G$1.2Z
- net VRED: now also U1.A; no longer IC1G$1.1Z
Other:
- moved on the sheet: R7, R9

Commit message: Cleanup
Other:
- moved on the sheet: R7, R8, R9, U1, X1-1, X1-10, X1-11, X1-12, X1-13, X1-14, X1-15, X1-2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
