File: breakout/breakout.brd (EAGLE design)
At the start: 20 x 19 mm, 4 parts, among them J1 DIN13T

Commit message: Breakout, logical placement of the headers
Parts:
- turned JP2 to 90 degrees
Routing:
- net N$12: track 13.5 -> 21.3 mm, vias 1 -> 0
- net N$8: track 13.4 -> 19.9 mm, vias 0 -> 1
- net N$11: track 9.84 -> 13.8 mm
- net N$10: track 8.17 -> 11.4 mm
- net N$5: track 13.4 -> 15.9 mm
- net N$6: track 12.2 -> 13.4 mm
- net N$9: track 5.85 -> 4.81 mm
- net N$2: track 9.84 -> 10.7 mm
- net N$7: track 12.2 -> 12.9 mm
- net N$3: track 8.20 -> 8.88 mm
- net N$1: track 13.7 -> 13.5 mm, vias 1 -> 0
Other:
- board text added: "Mono"
- board text removed: "Monochrome"

Commit message: Why not group things together?
Parts:
- moved JP3 15.2 mm to (10.0, 4.92)
- moved J1 1.27 mm to (10.0, 12.5)
- moved JP1 1.27 mm to (1.95, 12.5)
- moved JP2 1.27 mm to (18.1, 12.5), turned to 270 degrees
Connections:
- removed net N$6 (its old number): J1.6, JP1.6
- new net N$7: J1.6, JP2.2
- net N$10: now also J1.11, JP2.6; no longer J1.10, JP2.4
- net N$11: now also J1.9, JP2.4; no longer J1.11, JP2.5
- net N$12: now also JP2.5; no longer JP2.6
- net N$8: now also JP1.6; no longer JP2.2
- net N$9: now also J1.10; no longer J1.9
Routing:
- net N$6 (its old number): track 13.4 -> 0.00 mm
- net N$8: track 19.9 -> 8.13 mm, vias 1 -> 0
- net N$11: track 13.8 -> 4.84 mm
- net N$12: track 21.3 -> 12.5 mm
- net N$7: track 0.00 -> 8.42 mm
- net N$9: track 4.81 -> 8.37 mm
- net N$5: track 15.9 -> 13.4 mm
- net N$3: track 8.88 -> 7.34 mm
- net N$2: track 10.7 -> 9.84 mm
- net N$6: track 12.9 -> 12.2 mm
- net N$10: track 11.4 -> 10.9 mm
Other:
- board size 20 x 19 mm -> 20 x 17.5 mm
