File: mk5.1/SMD.brd (EAGLE design)
At the start: 31.9 x 37.7 mm, 9 parts, among them IC2 78L05F

Commit message: BEtter placement of TS5V330
Parts:
- moved IC2 15.5 mm to (16.9, 29.7)
- moved TS5V330 11.6 mm to (27.6, 20.6), flipped to the bottom, turned to 270 degrees
- moved S1 1.27 mm to (31.1, 29.3)
Routing:
- net GOUT: track 6.69 -> 63.4 mm, vias 0 -> 1
- net VGREEN: track 58.2 -> 14.6 mm
- net +5V: track 35.9 -> 18.1 mm
- net BOUT: track 17.3 -> 33.0 mm
- net VBLUE: track 24.4 -> 10.9 mm
- net AMONO: track 39.8 -> 26.6 mm, vias 3 -> 0
- net ARED: track 33.9 -> 22.9 mm
- net MONODETECT: track 11.9 -> 21.9 mm
- net ABLUE: track 33.4 -> 25.4 mm
- net ROUT: track 8.56 -> 15.6 mm
- net VRED: track 23.9 -> 17.0 mm
- net VCC: track 7.77 -> 12.7 mm
- net AAUDIO: track 17.5 -> 21.4 mm, vias 1 -> 0
- net AGREEN: track 21.7 -> 20.6 mm
- net SELECT: track 6.19 -> 5.50 mm, vias 0 -> 1
