File: mk6/mk6.brd (EAGLE design)
At the start: 31.3 x 34.7 mm, 11 parts, among them IC2 78L05F, U1 ATTINY85-20SU

Commit message: 'Trying to do things properly often comes back to haunt you' - Exxos. Moved a via that could mess things up. Modified the footprint of the button to make it easier when soldering.
Routing:
- net N$5: track 13.2 -> 14.6 mm
Changed lines of the file:
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@@
 <?xml version="1.0" encoding="utf-8"?>
 <!DOCTYPE eagle SYSTEM "eagle.dtd">
-<eagle version="8.2.0">
+<eagle version="8.3.0">
 <drawing>
 <settings>
 <setting alwaysvectorfont="no"/>
+<setting keepoldvectorfont="yes"/>
 <setting verticaltext="up"/>
 </settings>
@@
 <wire x1="11.43" y1="27.94" x2="11.43" y2="26.915" width="0.4064" layer="16"/>
 <wire x1="11.43" y1="26.915" x2="11.625" y2="26.72" width="0.4064" layer="16"/>
-<via x="17.78" y="32.512" extent="1-16" drill="0.3048"/>
-<via x="12.192" y="25.146" extent="1-16" drill="0.3048"/>
+<via x="22.733" y="31.496" extent="1-16" drill="0.3048"/>
+<via x="12.192" y="24.511" extent="1-16" drill="0.3048"/>
 </signal>
 <signal name="AGREEN">
@@
 <wire x1="9.144" y1="20.3835" x2="8.1915" y2="19.431" width="0.254" layer="1"/>
 <wire x1="9.144" y1="21.5265" x2="9.144" y2="20.3835" width="0.254" layer="1"/>
-<wire x1="9.7155" y1="22.098" x2="9.144" y2="21.5265" width="0.254" layer="1"/>
-<wire x1="9.906" y1="22.098" x2="9.7155" y2="22.098" width="0.254" layer="1"/>
-<wire x1="10.0965" y1="22.2885" x2="9.906" y2="22.098" width="0.254" layer="1"/>
-<wire x1="10.4775" y1="22.2885" x2="10.0965" y2="22.2885" width="0.254" layer="1"/>
-<wire x1="10.668" y1="22.479" x2="10.4775" y2="22.2885" width="0.254" layer="1"/>
-<wire x1="11.43" y1="22.479" x2="10.668" y2="22.479" width="0.254" layer="1"/>
-<wire x1="12.0015" y1="21.9075" x2="11.43" y2="22.479" width="0.254" layer="1"/>
-<wire x1="15.24" y1="21.9075" x2="12.0015" y2="21.9075" width="0.254" layer="1"/>
-<wire x1="16.9545" y1="23.622" x2="15.24" y2="21.9075" width="0.254" layer="1"/>
+<wire x1="9.144" y1="21.5265" x2="9.7155" y2="22.098" width="0.254" layer="1"/>
 <wire x1="21.5265" y1="23.622" x2="16.9545" y2="23.622" width="0.254" layer="16"/>
 <wire x1="23.4315" y1="21.717" x2="21.5265" y2="23.622" width="0.254" layer="16"/>
@@
 <wire x1="22.2885" y1="19.05" x2="22.21" y2="18.9" width="0.254" layer="16"/>
 <via x="16.9545" y="23.622" extent="1-16" drill="0.3048"/>
+<wire x1="11.496775" y1="22.098" x2="12.332175" y2="22.9334" width="0.254" layer="1"/>
+<wire x1="9.7155" y1="22.098" x2="11.496775" y2="22.098" width="0.254" layer="1"/>
+<wire x1="16.2659" y1="22.9334" x2="16.9545" y2="23.622" width="0.254" layer="1"/>
+<wire x1="12.332175" y1="22.9334" x2="16.2659" y2="22.9334" width="0.254" layer="1"/>
 </signal>
 <signal name="ARED">
@@
 <contactref element="TS5V330" pad="11"/>
 <contactref element="TM3" pad="2"/>
-<wire x1="7.8105" y1="17.145" x2="7.8105" y2="16.383" width="0.254" layer="1"/>
-<wire x1="9.144" y1="18.4785" x2="7.8105" y2="17.145" width="0.254" layer="1"/>
-<wire x1="9.144" y1="19.05" x2="9.144" y2="18.4785" width="0.254" layer="1"/>
-<wire x1="8.9535" y1="19.2405" x2="9.144" y2="19.05" width="0.254" layer="1"/>
-<wire x1="8.9535" y1="19.6215" x2="8.9535" y2="19.2405" width="0.254" layer="1"/>
-<wire x1="9.525" y1="20.193" x2="8.9535" y2="19.6215" width="0.254" layer="1"/>
-<wire x1="9.525" y1="21.1455" x2="9.525" y2="20.193" width="0.254" layer="1"/>
-<wire x1="10.287" y1="21.9075" x2="9.525" y2="21.1455" width="0.254" layer="1"/>
-<wire x1="11.049" y1="21.9075" x2="10.287" y2="21.9075" width="0.254" layer="1"/>
-<wire x1="11.049" y1="23.0505" x2="11.049" y2="21.9075" width="0.254" layer="16"/>
-<wire x1="12.7635" y1="24.765" x2="11.049" y2="23.0505" width="0.254" layer="16"/>
-<wire x1="12.7635" y1="26.67" x2="12.7635" y2="24.765" width="0.254" layer="16"/>
-<wire x1="7.8105" y1="16.383" x2="7.8" y2="16.24" width="0.254" layer="1"/>
-<wire x1="12.7635" y1="26.67" x2="12.895" y2="26.72" width="0.254" layer="16"/>
-<via x="11.049" y="21.9075" extent="1-16" drill="0.3048"/>
+<wire x1="7.8" y1="16.24" x2="7.8105" y2="16.383" width="0.254" layer="1"/>
+<wire x1="12.895" y1="26.72" x2="12.7635" y2="26.67" width="0.254" layer="16"/>
+<wire x1="13.081" y1="25.527" x2="13.462" y2="25.146" width="0.254" layer="16"/>
+<wire x1="13.081" y1="25.527" x2="13.081" y2="26.534" width="0.254" layer="16"/>
+<wire x1="13.081" y1="26.534" x2="12.895" y2="26.72" width="0.254" layer="16"/>
+<via x="13.462" y="21.971" extent="1-16" drill="0.35"/>
+<wire x1="13.462" y1="25.146" x2="13.462" y2="21.971" width="0.254" layer="16"/>
+<wire x1="13.462" y1="21.971" x2="13.462" y2="19.685" width="0.254" layer="1"/>
+<wire x1="13.462" y1="19.685" x2="12.192" y2="18.415" width="0.254" layer="1"/>
+<wire x1="12.192" y1="18.415" x2="9.975" y2="18.415" width="0.254" layer="1"/>
+<wire x1="9.975" y1="18.415" x2="7.8" y2="16.24" width="0.254" layer="1"/>
 </signal>
 <signal name="AUDIOPOT">
@@
 <wire x1="23.0505" y1="33.147" x2="26.0985" y2="30.099" width="0.254" layer="1"/>
 <wire x1="27.051" y1="26.67" x2="27.157896875" y2="26.648728125" width="0.254" layer="16"/>
-<wire x1="23.0505" y1="33.147" x2="22.91" y2="33.21" width="0.254" layer="1"/>
+<wire x1="23.0505" y1="33.147" x2="23.2148" y2="33.21" width="0.254" layer="1"/>
 <via x="26.0985" y="27.432" extent="1-16" drill="0.3048"/>
 </signal>
